File: kicad/hiki/hiki.kicad_sch (KiCad schematic)
At the start: 2 parts

Commit message: check point
Parts:
- added J1: Screw_Terminal_01x02, symbol Connector:Screw_Terminal_01x02
- added SW1: SW_SPDT, symbol hiki:SW_SPDT
- added Z1: Power Supply Unit, symbol Mechanical:Housing
- added Z2: Battery Assembly, symbol Device:Battery_Cell
Connections:
- net GND: now also J1.2 (Pin_2)
- net +5V: no longer names the net of R1.1
- net +5V: now also SW1.2 (on)
- new net VCC: J1.1 (Pin_1), SW1.3 (common)
Other:
- moved on the sheet: D1, R1

Commit message: finish schematic
Connections:
- no-connect marks 0 -> 3
Other:
- moved on the sheet: Z1, Z2

Commit message: save befor adding footprint lib
Parts:
- D1: footprint (none) -> LED_THT:LED_D5.0mm
- J1: footprint (none) -> TerminalBlock_Phoenix:TerminalBlock_Phoenix_PT-1,5-2-5.0-H_1x02_P5.00mm_Horizontal
- R1: footprint (none) -> Resistor_THT:R_Axial_DIN0207_L6.3mm_D2.5mm_P7.62mm_Horizontal
Changed lines of the file:
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@@
 			)
 		)
-		(property "Footprint" ""
+		(property "Footprint" "LED_THT:LED_D5.0mm"
 			(at 162.56 83.82 0)
 			(hide yes)
@@
 			)
 		)
-		(property "Footprint" ""
+		(property "Footprint" "Resistor_THT:R_Axial_DIN0207_L6.3mm_D2.5mm_P7.62mm_Horizontal"
 			(at 151.13 83.82 0)
 			(hide yes)
@@
 			)
 		)
-		(property "Footprint" ""
+		(property "Footprint" "TerminalBlock_Phoenix:TerminalBlock_Phoenix_PT-1,5-2-5.0-H_1x02_P5.00mm_Horizontal"
 			(at 111.76 82.55 0)
 			(hide yes)

Commit message: finish footprint assignments
Parts:
- SW1: footprint (none) -> hiki:SWITCH_SPDT_3P
Changed lines of the file:
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@@
 			)
 		)
-		(property "Footprint" ""
+		(property "Footprint" "hiki:SWITCH_SPDT_3P"
 			(at 135.89 82.55 0)
 			(hide yes)
