File: kicad/hiki/hiki.kicad_pcb (KiCad board)
At the start: 2 copper layers, 4 parts, among them J1 Screw_Terminal_01x02, SW1 SW_SPDT

Commit message: done with pcb
Parts:
- added REF**: MountingHole_3.2mm_M3, MountingHole:MountingHole_3.2mm_M3, F.Cu at (186.0, 74.2)
- added REF**: MountingHole_3.2mm_M3, MountingHole:MountingHole_3.2mm_M3, F.Cu at (114.0, 74.1)
- added REF**: MountingHole_3.2mm_M3, MountingHole:MountingHole_3.2mm_M3, F.Cu at (113.5, 126.2)
- added REF**: MountingHole_3.2mm_M3, MountingHole:MountingHole_3.2mm_M3, F.Cu at (186.3, 126.0)
- moved J1 16.5 mm to (121.3, 88.3)
- moved D1 16.5 mm to (183.6, 100.8)
- moved R1 16.5 mm to (159.6, 98.3)
- moved SW1 16.5 mm to (149.5, 98.3)
Routing:
- net GND: track 85.3 -> 0.00 mm
- net VCC: track 28.2 -> 0.01 mm
- added copper zone on F.Cu, net GND
- added copper zone on B.Cu, net VCC
Other:
- board outline added: 155.2 x 86.9 mm
